Commit message: collision

File: assets/base_objects/clamps.urdf (robot description, URDF)
Before this commit: robot panda_clamps.urdf, 2 links, 1 joints
Links:
- removed link panda_clamps_link
- added link clamps_link, mass 0.112; collision box size=0.06985 0.19685 0.20955; visual box size=0.06985 0.19685 0.20955
Joints:
- joint clamps_joint: child panda_clamps_link -> clamps_link

File: assets/base_objects/support_beams.urdf (robot description, URDF)
Before this commit: robot panda_support_beams.urdf, 2 links, 1 joints
Links:
- removed link panda_support_beam_link
- added link support_beam_link, mass 0.112; collision box size=0.3048 0.19685 0.04445; visual box size=0.3048 0.19685 0.04445
Joints:
- joint support_joint: child panda_support_beam_link -> support_beam_link
