Commit message: remove joints from urdfs

File: assets/base_objects/back_wall.urdf (robot description, URDF)
Before this commit: robot wall.urdf, 2 links, 1 joints
Links:
- removed link world
Joints:
- removed joint wall_joint

File: assets/base_objects/clamps.urdf (robot description, URDF)
Before this commit: robot clamps.urdf, 2 links, 1 joints
Links:
- removed link world
Joints:
- removed joint clamps_joint

File: assets/base_objects/plane.urdf (robot description, URDF)
Before this commit: robot plane, 2 links, 1 joints
Links:
- removed link world
Joints:
- removed joint plane_joint

File: assets/base_objects/support_beams.urdf (robot description, URDF)
Before this commit: robot support_beams.urdf, 2 links, 1 joints
Links:
- removed link world
Joints:
- removed joint support_joint

File: assets/base_objects/table_ikea.urdf (robot description, URDF)
Before this commit: robot table_ikea.urdf, 2 links, 1 joints
Links:
- removed link world
Joints:
- removed joint table_ikea_joint

File: assets/base_objects/table_wooden.urdf (robot description, URDF)
Before this commit: robot table_wooden.urdf, 2 links, 1 joints
Links:
- removed link world
Joints:
- removed joint table_wooden_joint
